File: mm_motor_control.kicad_sch (KiCad schematic)
At the start: 0 parts

Commit message: fin tp2
Parts:
- added C7, Cstby: 1nF, symbol Device:C
- added Crcoff: 22nF, symbol Device:C
- added Cs, Cspol: 22uF, symbol Device:C
- added R, R11: 2.2K, symbol Device:R
- added R10: 18K, symbol Device:R
- added Roff: 47K, symbol Device:R
- added Rrcoff: 1K, symbol Device:R
- added Rsnsb, Rsnsb1: 330m, symbol Device:R
- added Rstby: 10K, symbol Device:R
- added U2: STSPIN240, Package_DFN_QFN:VQFN-16-1EP_3x3mm_P0.5mm_EP1.8x1.8mm, symbol Driver_Motor:STSPIN240
Connections:
- net EN: now also C7.2, R10.2, U2.13 (EN/FLT)
- net FAULT: now also R10.1
- net OUT_A1: now also U2.3 (OUTA1)
- net OUT_A2: now also U2.5 (OUTA2)
- net OUT_B1: now also U2.10 (OUTB1)
- net OUT_B2: now also U2.8 (OUTB2)
- net PHASE_A: now also U2.1 (PHA)
- net PHASE_B: now also U2.15 (PHB)
- net PWM_A: now also U2.2 (PWMA)
- net STBY/RESET: now also Cstby.2, Rstby.1, U2.14 (STBY/RESET)
- new net: R.2, R11.1, U2.11 (REF)
- new net: Roff.1, Rrcoff.1, U2.12 (TOFF)
- new net: Crcoff.2, Rrcoff.2
- new net: Rsnsb1.1, U2.4 (SENSEA)
- new net: Rsnsb.1, U2.9 (SENSEB)
- new net +BATT: R11.2
- new net GND: C7.1, Crcoff.1, Cs.2, Cspol.1, Cstby.1, R.1, Roff.2, Rsnsb.2, Rsnsb1.2, U2.16 (PWMB), U2.17 (EPAD), U2.7 (GND)
- new net VDD: Rstby.2
- new net VS: Cs.1, Cspol.2, U2.6 (VS)

Commit message: TP3
Parts:
- removed C7, Cstby: 1nF, symbol Device:C
- removed Cs, Cspol: 22uF, symbol Device:C
- removed R10: 18K, symbol Device:R
- removed Rsnsb1: 330m, symbol Device:R
- removed Rstby: 10K, symbol Device:R
- added C11: 1nF, Capacitor_SMD:C_0603_1608Metric, symbol Device:C
- added C12: 2.2uF, Capacitor_SMD:C_0603_1608Metric, symbol Device:C
- added R12: 330m, Resistor_SMD:R_0603_1608Metric, symbol Device:R
- added R17: 10K, Resistor_SMD:R_0603_1608Metric, symbol Device:R
- C10: renamed from Crcoff; footprint (none) -> Capacitor_SMD:C_0603_1608Metric
- R11: renamed from Rsnsb; footprint (none) -> Resistor_SMD:R_0603_1608Metric
- R13: renamed from R11; value 2.2K -> 10K; footprint (none) -> Resistor_SMD:R_0603_1608Metric
- R14: renamed from R; value 2.2K -> 10K; footprint (none) -> Resistor_SMD:R_0603_1608Metric
- R15: renamed from Rrcoff; footprint (none) -> Resistor_SMD:R_0603_1608Metric
- R16: renamed from Roff; footprint (none) -> Resistor_SMD:R_0603_1608Metric
- renumbered U2 to U3
Connections:
- net VS is gone; now on net +BATT: U3.6 (VS)
- net +BATT: now also C12.1
- net EN: now also R17.1; no longer U3.13 (EN/FLT)
- net FAULT: now also U3.13 (EN/FLT), C11.1, R17.2
- net GND: now also C11.2, C12.2, R12.2; no longer U3.16 (PWMB)
- net at U3.4 (SENSEA): now also R12.1
- new net PWM_B: U3.16 (PWMB)
