File: tp2cao.kicad_pcb (KiCad board)
At the start: 2 copper layers, 90 x 85 mm, 50 parts, among them J1 Conn_ARM_JTAG_SWD_10, J2 Conn_01x04, J4 Conn_01x06, J5 Conn_01x02, J6 Conn_01x06, M1 N20_encoder, M2 N20_encoder, U1 STM32F030C8Tx, U2 LP5907MFX-1.2, U3 STSPIN240, U4 HC-SR04

Commit message: TP4
Parts:
- moved C13 56.1 mm to (171.8, 84.8), turned to -90 degrees
- moved C14 50.5 mm to (130.9, 102.5)
- moved C9 49.7 mm to (186.7, 84.5), turned to -90 degrees
- moved R11 44.0 mm to (153.9, 102.8)
- moved R18 43.8 mm to (188.8, 80.7), turned to -90 degrees
- moved C7 42.0 mm to (120.8, 75.0), turned to 180 degrees
- moved U3 36.7 mm to (146.4, 101.2)
- moved R10 35.8 mm to (129.7, 77.5), turned to 180 degrees
- moved R9 33.2 mm to (145.7, 75.0)
- moved R20 32.4 mm to (126.1, 92.9), turned to -90 degrees
- moved R1 31.0 mm to (147.3, 75.0)
- moved R12 30.1 mm to (142.3, 102.1), turned to 180 degrees
- moved C15 28.9 mm to (153.8, 72.6), turned to -90 degrees
- moved R19 28.5 mm to (170.4, 91.7), turned to 180 degrees
- moved D1 27.7 mm to (188.8, 84.3), turned to 90 degrees
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Routing:
- net +BATT: track 0.00 -> 68.6 mm
- net +3.3V: track 0.00 -> 52.1 mm
- net GND: track 0.00 -> 38.1 mm, vias 0 -> 24
- net Net-(U3-REF): track 0.00 -> 10.5 mm
- net /mcu/IN_B2: track 0.00 -> 9.22 mm
- net Net-(J6-Pin_3): track 0.00 -> 6.78 mm
- net Net-(J6-Pin_4): track 0.00 -> 6.57 mm
- net Net-(U3-TOFF): track 0.00 -> 5.84 mm
- net Net-(U3-SENSEB): track 0.00 -> 5.65 mm
- net Net-(U1-PA2): track 0.00 -> 5.33 mm
- net Net-(J4-Pin_4): track 0.00 -> 4.79 mm
- net Net-(J4-Pin_3): track 0.00 -> 4.76 mm
- net Net-(U1-PB9): track 0.00 -> 4.42 mm
- net /mcu/BOOT0: track 0.00 -> 4.16 mm
- net Net-(U1-PB6): track 0.00 -> 3.98 mm
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- added copper zone on B.Cu, net GND

Commit message: TP5
Parts:
- moved C5 39.0 mm to (141.4, 75.5), turned to 90 degrees
- moved R21 24.7 mm to (148.8, 91.7), turned to -90 degrees
- moved J4 12.5 mm to (130.2, 90.3), turned to 0 degrees
- moved R18 12.4 mm to (176.9, 76.9)
- moved R17 10.7 mm to (153.5, 91.6)
- moved C3 10.6 mm to (137.2, 85.6)
- moved D1 9.92 mm to (180.2, 79.2)
- moved R19 8.78 mm to (164.8, 98.5), turned to -90 degrees
- moved C9 6.77 mm to (180.0, 83.8)
- moved U2 6.77 mm to (174.7, 81.0)
- moved C8 6.76 mm to (169.6, 80.4), turned to 90 degrees
- moved C10 6.74 mm to (153.1, 101.6)
- moved C11 6.74 mm to (147.9, 101.6)
- moved R15 6.74 mm to (151.4, 101.6)
- moved R16 6.74 mm to (149.7, 101.6)
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Connections:
- C12 pad 1: +BATT -> /motorB/MB
- J1 pad 2: /mcu/SWDIO -> +3.3V
- J1 pad 4: /mcu/SWDCLK -> +3.3V
- J5 pad 2: +BATT -> /motorB/MB
- J6 pad 5: +BATT -> /motorB/MB
- R11 pad 1: Net-(U3-SENSEB) -> /motorB/MB
- R13 pad 2: +BATT -> /motorB/MB
- R16 pad 2: GND -> /motorB/MB
- R17 pad 1: /mcu/OUT_B1 -> +3.3V
- R17 pad 2: /mcu/IN_B2 -> +3.3V
- R2 pad 2: /mcu/TIM15_CH1 -> /motorB/MA
- R7 pad 1: /mcu/OUT_B1 -> +3.3V
- R7 pad 2: Net-(U1-PB1) -> +3.3V
- U1 pad 19: Net-(U1-PB1) -> +3.3V
- U1 pad 20: /mcu/IN_B2 -> +3.3V
- U1 pad 21: unconnected-(U1-PB10-Pad21) -> +3.3V
- U1 pad 22: unconnected-(U1-PB11-Pad22) -> +3.3V
- U1 pad 23: GND -> +3.3V
- U1 pad 33: unconnected-(U1-PA12-Pad33) -> +3.3V
- U1 pad 34: /mcu/SWDIO -> +3.3V
- U1 pad 35: unconnected-(U1-PF6-Pad35) -> +3.3V
- U1 pad 37: /mcu/SWDCLK -> +3.3V
- U3 pad 1: /mcu/OUT_A4 -> /motorB/MA
- U3 pad 10: /motorA/MA -> /motorB/MB
- U3 pad 13: /mcu/IN_B2 -> +3.3V
- U3 pad 2: /mcu/TIM15_CH1 -> /motorB/MA
- U3 pad 4: Net-(U3-SENSEA) -> /motorB/MA
- U3 pad 6: +BATT -> /motorB/MB
- U3 pad 7: GND -> /motorB/MB
- U3 pad 9: Net-(U3-SENSEB) -> /motorB/MB
Routing:
- net /motorB/MB: track 0.00 -> 114.4 mm, vias 0 -> 1
- net +3.3V: track 52.1 -> 107.7 mm
- net +BATT: track 68.6 -> 40.4 mm
- net /mcu/TIM2_CH1: track 0.00 -> 26.2 mm
- net /mcu/TIM2_CH2: track 0.00 -> 23.7 mm
- net /mcu/TIM8_CH2: track 0.00 -> 23.4 mm
- net /motorB/MA: track 0.00 -> 22.0 mm
- net /mcu/SWO: track 0.00 -> 12.4 mm
- net /mcu/BOOT0: track 4.16 -> 15.1 mm
- net /mcu/IN_B2: track 9.22 -> 0.00 mm
- net Net-(J4-Pin_3): track 4.76 -> 11.9 mm
- net /mcu/OUT_B9: track 0.00 -> 6.25 mm
- net /mcu/OUT_A5: track 0.00 -> 5.72 mm
- net Net-(U3-SENSEB): track 5.65 -> 0.00 mm
- net /mcu/OUT_B0: track 0.00 -> 4.65 mm
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